File: IO_Board.kicad_sch (KiCad schematic)
At the start: 6 parts, among them CN301 SM32B-NSHDZS-1-TF, CN302 SM32B-NSHDZS-1-TF

Commit message: JLCPCB: W2026061412450502 2026-06-14 PCB: Y62-5297522A PCBA: SMT026061460215-5297522A
Parts:
- added +V1, +V5, +V7, +V9: +3V3, symbol My Power Management:+V (Local)
- added +V10, +V2, +V3, +V8: +V_{BAT}, symbol My Power Management:+V (Local)
- added +V4, +V6: +5V_{FUSED}, symbol My Power Management:+V (Local)
- added GND1, GND2, GND3, GND4, GND5, GND6: GND, symbol My Power Management:GND (Local)
- CN301, CN302: symbol PersonalSchematicSymbolLibrary:Conn_02x16_Odd_Even_MountingPin -> PersonalSchematicSymbolLibrary:Conn_02x16_Odd_Even_2MountingPins
- U301: renamed from U201; now left out of the parts list
Connections:
- net +3V3: now also +V1.1, +V5.1, +V7.1, +V9.1
- net +5V_{FUSED}: now also +V4.1, +V6.1
- net +V_{BAT}: now also +V10.1, +V2.1, +V3.1, +V8.1
- net GND: now also CN301.MP2 (MountPin), CN302.MP1 (MountPin), CN302.MP2 (MountPin), GND1.1 (GND), GND2.1 (GND), GND3.1 (GND), GND4.1 (GND), GND5.1 (GND), GND6.1 (GND); no longer CN301.MP (MountPin), CN302.MP (MountPin)
- net RLY-: now also CN301.MP1 (MountPin)
- net +5V_{EXT}: no longer names the net of U301.28 (+5V_{EXT})
- net IO00: no longer names the net of U301.12 (IO00)
- net IO01: no longer names the net of U301.3 (IO01)
- net IO03: no longer names the net of U301.4 (IO03)
- net IO45: no longer names the net of U301.22 (IO45)
- net IO46: no longer names the net of U301.21 (IO46)
- no-connect marks 0 -> 6
Other:
- sheet CAN Bus ports: added +3V3, +V_{BAT}, GND; removed none
- sheet GR86 Inputs ports: added +3V3, +5V_{FUSED}, GND; removed none
- sheet WLED Outputs ports: added +3V3, +5V_{FUSED}, +V_{BAT}, GND; removed none
